Commit message: Make a simulation acquisition automater.

File: intrinsic_simulation/urdf/target.urdf (robot description, URDF)
Before this commit: robot simple_camera, 4 links, 3 joints
Joints:
- joint sled_head_joint: origin xyz=${sled_xyz} rpy=${sled_rpy} -> xyz=$(arg sled_xyz) rpy=$(arg sled_rpy)
