Commit message: Made camera behavior parametrizable.

File: intrinsic_simulation/urdf/camera.urdf (robot description, URDF)
Before this commit: robot simple_camera, 3 links, 2 joints
Joints:
- joint camera_optical_joint_real: origin xyz=-0.102 0.017 -0.4 rpy=0 0 0 -> xyz=${yml_dict['x']} ${yml_dict['y']} ${yml_dict['z']} rpy=${yml_dict['r']} ${yml_dict['p']} ${yml_dict['w']}

Commit message: Frame terminology fixup.

File: intrinsic_simulation/urdf/camera.urdf (robot description, URDF)
Before this commit: robot simple_camera, 3 links, 2 joints
Joints:
- joint camera_optical_joint_real: origin xyz=${yml_dict['x']} ${yml_dict['y']} ${yml_dict['z']} rpy=${yml_dict['r']} ${yml_dict['p']} ${yml_dict['w']} -> xyz=${yml_dict['mill_to_camera_x']} ${yml_dict['mill_to_camera_y']} ${yml_dict['mill_to_camera_z']} rpy=${yml_dict['mill_to_camera_r']} ${yml_dict['mill_to_camera_p']} ${yml_dict['mill_to_camera_w']}

Commit message: Switch camera plugin to CWRU version.

File: intrinsic_simulation/urdf/camera.urdf (robot description, URDF)
Before this commit: robot simple_camera, 3 links, 2 joints
Links:
- removed link camera_optical_link_fixed
Joints:
- removed joint camera_optical_joint_fixed
