Commit message: Improve speed and stability of simulated target placement routine.

File: intrinsic/intrinsic_simulation/urdf/target.urdf (robot description, URDF)
Before this commit: robot simple_camera, 4 links, 3 joints
Links:
- removed link world
Joints:
- removed joint sled_head_joint

Commit message: Fix yaw transform.

File: intrinsic/intrinsic_simulation/urdf/target.urdf (robot description, URDF)
Before this commit: robot simple_camera, 3 links, 2 joints
Joints:
- joint sled_head_to_target_joint: origin xyz=     ${yml_dict_position['sled_to_target_x']}     ${yml_dict_position['sled_to_target_y']}     ${yml_dict_position['sled_to_target_z']}     rpy=     ${yml_dict_position['sled_to_target_r']}     ${yml_dict_position['sled_to_target_p']}     ${yml_dict_position['sled_to_target_y']}     -> xyz=     ${yml_dict_position['sled_to_target_x']}     ${yml_dict_position['sled_to_target_y']}     ${yml_dict_position['sled_to_target_z']}     rpy=     ${yml_dict_position['sled_to_target_r']}     ${yml_dict_position['sled_to_target_p']}     ${yml_dict_position['sled_to_target_w']}    
