Commit message: Work with two cameras.

File: intrinsic/intrinsic_simulation/urdf/camera.urdf (robot description, URDF)
Before this commit: robot simple_camera, 2 links, 1 joints
Links:
- removed link camera_optical_link_real
- added link camera_optical_link_left, mass 1e-5; visual box size=0.001 0.001 0.001
- added link camera_optical_link_right, mass 1e-5; visual box size=0.001 0.001 0.001
Joints:
- removed joint camera_optical_joint_real
- added joint camera_optical_joint_left: type fixed, parent world, child camera_optical_link_left, origin xyz=${yml_dict_1['mill_to_camera_x']} ${yml_dict_1['mill_to_camera_y']} ${yml_dict_1['mill_to_camera_z']} rpy=${yml_dict_1['mill_to_camera_r']} ${yml_dict_1['mill_to_camera_p']} ${yml_dict_1['mill_to_camera_w']}
- added joint camera_optical_joint_right: type fixed, parent world, child camera_optical_link_right, origin xyz=${yml_dict_2['mill_to_camera_x']} ${yml_dict_2['mill_to_camera_y']} ${yml_dict_2['mill_to_camera_z']} rpy=${yml_dict_2['mill_to_camera_r']} ${yml_dict_2['mill_to_camera_p']} ${yml_dict_2['mill_to_camera_w']}
